File: PCB/PowerSupply/bacteroid-PowerSupply.sch (KiCad schematic (older format))
At the start: 15 parts, among them P1 CONN_2, P2 CONN_2, P3 CONN_4, U1 LM7805CT, U2 LM7805CT, U3 LM7809CT, U4 LM7812CT

Commit message: PCB Updates
Parts:
- added R1, R2, R3: 0R, ~, symbol R
Connections:
- net +24V: now also R1.1, R2.1; no longer C1.1, C2.1, C4.1, U1.1 (IN), U2.1 (IN), U4.1 (IN)
- new net: C1.1, R3.2, U1.1 (IN)
- new net: C2.1, R1.2, R3.1, U2.1 (IN)
- new net: C4.1, R2.2, U4.1 (IN)
Other:
- moved on the sheet: C1, C5, P1, P2, U1
