File: PCB/DualMotorControl_1/bacteroid-DualMotorControl_1.kicad_pcb (KiCad board)
At the start: 2 copper layers, 35 parts, among them IC1 L298, P1 CONN_3X2, P2 CONN_8X2, P3 CONN_8X2, P4 CONN_8X2, Q1 PUMH9, Q2 PUMH9, Q3 PUMH9, U1 SN74HC14

Commit message: PCB update
Connections:
- D1 pad 1: N-0000036 (its old number) -> GND
- D1 pad 2: N-0000035 (its old number) -> N-0000033
- D2 pad 1: N-0000034 (its old number) -> GND
- D3 pad 1: N-0000033 -> GND
- D3 pad 2: N-0000030 (its old number) -> N-0000028
- D4 pad 1: N-0000020 -> GND
- D5 pad 1: N-0000035 (its old number) -> N-0000033
- D7 pad 1: N-0000030 (its old number) -> N-0000028
- IC1 pad 13: N-0000033 -> N-0000028
- IC1 pad 14: N-0000020 -> N-0000032
- IC1 pad 2: N-0000036 (its old number) -> N-0000033
- IC1 pad 3: N-0000034 (its old number) -> N-0000029
- P4 pad 1: N-0000035 (its old number) -> N-0000033
- P4 pad 10: N-0000030 (its old number) -> N-0000028
- P4 pad 11: N-0000030 (its old number) -> N-0000028
- P4 pad 12: N-0000030 (its old number) -> N-0000028
- P4 pad 2: N-0000035 (its old number) -> N-0000033
- P4 pad 3: N-0000035 (its old number) -> N-0000033
- P4 pad 4: N-0000035 (its old number) -> N-0000033
- P4 pad 9: N-0000030 (its old number) -> N-0000028
