File: PCB/DualMotorControl_1/bacteroid-DualMotorControl_1.sch (KiCad schematic (older format))
At the start: 31 parts

Commit message: PCB update
Parts:
- removed C?: C, ~, symbol C
- removed U? (x2): L298, MODULE, symbol L298
- added C3: 100nF, ~, symbol C
- added IC1: L298, st-microelectronics-MULTIWATT-15, symbol L298
- added JP1, JP2, JP3, JP4: JUMPER, ~, symbol JUMPER
- added JP5, JP6, JP7, JP8: JUMPER3, ~, symbol JUMPER3
- added P1: CONN_3X2, symbol CONN_3X2
- added P2, P3, P4: CONN_8X2, symbol CONN_8X2
- added R7: 10k, ~, symbol R
- C1, C2: renamed from C?; value C -> 100nF
- D1, D2, D3, D4, D5, D6, D7, D8: renamed from D?; value DIODE -> ES2DA
- R1, R2, R3, R4, R5, R6: renamed from R?; value R -> 10k
- U1: renamed from U?; value 74HC14 -> SN74HC14
- gave numbers to parts that had none: 3
Connections:
- net DRV1_EN1: now also P2.5
- net DRV1_EN1_TTL: now also U1.6, IC1.6 (ENABLE_A), P3.11; no longer U1.2
- net DRV1_EN2: now also Q3.5 (B), P2.6; no longer Q3.2 (B)
- net DRV1_EN2_TTL: now also U1.12, IC1.11 (ENABLE_B), JP2.1, P3.13; no longer U1.2
- net DRV1_IN1: now also P2.1
- net DRV1_IN1_TTL: now also JP1.1, P3.1
- net DRV1_IN2: now also Q1.5 (B), P2.2; no longer Q1.2 (B)
- net DRV1_IN2_TTL: now also U1.4, P3.3; no longer U1.2
- net DRV1_IN3: now also Q2.5 (B), P2.3; no longer Q2.2 (B)
- net DRV1_IN3_TTL: now also U1.8, JP3.1, P3.5; no longer U1.2
- net DRV1_IN4: now also P2.4
- net DRV1_IN4_TTL: now also U1.10, JP4.1, P3.7; no longer U1.2
- net GND: now also C1.2, C2.1, Q1.4 (E), Q2.4 (E), Q3.4 (E), C3.2, IC1.1 (SEN_A), IC1.15 (SEN_B), IC1.8 (GND), JP5.1, JP6.1, JP7.1, JP8.1, P2.10, P2.12, P2.14, P3.10, P3.12, P3.14, P3.16, P3.2, P3.4, P3.6, P3.8; no longer Q1.1 (E), Q2.1 (E), Q3.1 (E)
- net VCC: now also C1.1, C3.1, IC1.9 (VCC), P2.9, R7.1
- net at D1.1 (A): now also IC1.2 (OUT1)
- net at D1.2 (K): now also D5.1 (A), P4.1, P4.2, P4.3, P4.4
- net VSS: now reaches D5.2 (K)
- net VSS: now also C2.2, D6.2 (K), D7.2 (K), D8.2 (K), IC1.4 (VS), P1.2, P1.4, P1.6
- net at D2.1 (A): now also IC1.3 (OUT2)
- net at D2.2 (K): now also D6.1 (A), P4.5, P4.6, P4.7, P4.8
- net at D3.1 (A): now also IC1.13 (OUT3)
- net at D3.2 (K): now also D7.1 (A), P4.10, P4.11, P4.12, P4.9
- net at D4.1 (A): now also IC1.14 (OUT4)
- net at D4.2 (K): now also D8.1 (A), P4.13, P4.14, P4.15, P4.16
- net at Q2.6 (C), R3.2: now also U1.5; no longer U1.1
- net at Q3.6 (C), R5.2: now also U1.11; no longer U1.1
- new net: Q1.3 (C), R2.2, U1.3
- new net: Q2.3 (C), R4.2, U1.9
- new net: Q3.3 (C), R6.2, U1.13
- new net: IC1.10 (INPUT3), JP3.2, JP7.2
- new net: IC1.12 (INPUT4), JP4.2, JP8.2
- new net: IC1.5 (INPUT1), JP1.2, JP5.2
- new net: IC1.7 (INPUT2), JP2.2, JP6.2
- new net: JP5.3, JP6.3, JP7.3, JP8.3, R7.2
- new net +12V: P1.5, P2.16
- new net +5V: P1.1, P2.13
- new net +9V: P1.3, P2.15
- no-connect marks 0 -> 5
Other:
- note added: "1"
- note added: "BeagleBone TTL-Converter / Dual Motor Driver"
- moved on the sheet: C1, C2, D1, D2, D3, D4, D5, D6, D7, D8, Q1A, Q2A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

Commit message: PCB update
Connections:
- net GND: now also D1.1 (A), D2.1 (A), D3.1 (A), D4.1 (A)
- net at IC1.2 (OUT1): now also D1.2 (K), D5.1 (A), P4.1, P4.2, P4.3, P4.4; no longer D1.1 (A)
- net at IC1.3 (OUT2): now also D2.2 (K), D6.1 (A), P4.5, P4.6, P4.7, P4.8; no longer D2.1 (A)
- net at IC1.13 (OUT3): now also D3.2 (K), D7.1 (A), P4.10, P4.11, P4.12, P4.9; no longer D3.1 (A)
- net at IC1.14 (OUT4): now also D4.2 (K), D8.1 (A), P4.13, P4.14, P4.15, P4.16; no longer D4.1 (A)
Changed lines of the file:
@@
-EESchema Schematic File Version 2  date Sonntag, 06. Oktober 2013 17:10:19
+EESchema Schematic File Version 2  date Donnerstag, 10. Oktober 2013 21:19:51
 LIBS:power
 LIBS:device
@@
 Sheet 1 1
 Title ""
-Date "6 oct 2013"
+Date "10 oct 2013"
 Rev ""
 Comp ""
@@
 Wire Wire Line
 	9500 3450 9400 3450
-Wire Wire Line
-	8150 2500 8400 2500
-Wire Wire Line
-	8400 2500 8400 2250
-Wire Wire Line
-	8150 2600 8400 2600
-Wire Wire Line
-	8400 2600 8400 2850
-Wire Wire Line
-	8150 2400 8300 2400
-Wire Wire Line
-	8300 2400 8300 1650
-Wire Wire Line
-	8300 1650 8400 1650
-Wire Wire Line
-	8150 2700 8300 2700
-Wire Wire Line
-	8300 2700 8300 3450
-Wire Wire Line
-	8300 3450 8400 3450
 Connection ~ 9500 2250
 Connection ~ 9500 2850
@@
 	8900 1650 8900 1850
 Wire Wire Line
-	8900 1850 9700 1850
+	8850 1850 9700 1850
 Wire Wire Line
 	9700 1850 9700 2250
 Wire Wire Line
-	8900 2250 8900 2050
+	8900 2050 8900 2500
 Wire Wire Line
 	8900 2050 9600 2050
@@
 	8900 2850 8900 3050
 Wire Wire Line
-	8900 3050 9600 3050
+	8250 3050 9600 3050
 Wire Wire Line
 	9600 3050 9600 2650
@@
 	8900 3450 8900 3250
 Wire Wire Line
-	8900 3250 9700 3250
+	8200 3250 9700 3250
 Wire Wire Line
 	9700 3250 9700 2850
@@
 Wire Wire Line
 	3900 900  3900 1000
+$Comp
+L GND #PWR?
+U 1 1 5257010F
+P 8350 3600
+F 0 "#PWR?" H 8350 3600 30  0001 C CNN
+F 1 "GND" H 8350 3530 30  0001 C CNN
+F 2 "" H 8350 3600 60  0000 C CNN
+F 3 "" H 8350 3600 60  0000 C CNN
+	1    8350 3600
+	1    0    0    -1
+$EndComp
+Connection ~ 8900 3250
+Wire Wire Line
+	8150 2700 8200 2700
+Wire Wire Line
+	8200 2700 8200 3250
+Wire Wire Line
+	8400 3450 8350 3450
+Wire Wire Line
+	8350 1650 8350 3600
+Connection ~ 8900 3050
+Wire Wire Line
+	8150 2600 8250 2600
+Wire Wire Line
+	8250 2600 8250 3050
+Wire Wire Line
+	8900 2500 8150 2500
+Connection ~ 8900 1850
+Wire Wire Line
+	8150 2400 8850 2400
+Wire Wire Line
+	8850 2400 8850 1850
+Connection ~ 8350 3450
+Wire Wire Line
+	8400 1650 8350 1650
+Connection ~ 8350 2850
+Connection ~ 8350 2250
+Wire Wire Line
+	8400 2250 8350 2250
+Wire Wire Line
+	8400 2850 8350 2850
 $EndSCHEMATC
